File: cart_programmer/eng/kicad/cart_programmer/cart_programmer.kicad_pcb (KiCad board)
At the start: 2 copper layers, 7 parts, among them J1 CONN_ATARI_CART_PROGRAMMER, J2 CONN_ATARI_7800_CART_EDGE, K1 G5LE-1, U2 SFH617A-2

Commit message: Added Cartridge Programmer Serial Protocol Doc (WIP). Cartridge Programmer schematic (WIP). ROM/RAM/PLD Cartridge project skeleton.
Parts:
- J1: value CONN_ATARI_CART_PROGRAMMER -> CONN_512K_CART_SOCKET_PHY
- J2: value CONN_ATARI_7800_CART_EDGE -> CONN_A7K8_CART_CARD_PHY
Connections:
- D1 pad 1: Net-(D1-Pad1) -> (no net)
- D1 pad 2: Net-(D1-Pad2) -> (no net)
- D2 pad 1: Net-(D2-Pad1) -> (no net)
- D2 pad 2: Net-(D2-Pad2) -> (no net)
- J1 pad 1: /A1 -> (no net)
- J1 pad 10: /A10 -> (no net)
- J1 pad 11: /A11 -> (no net)
- J1 pad 12: Net-(J1-Pad12) -> (no net)
- J1 pad 13: /D0 -> (no net)
- J1 pad 14: /D2 -> (no net)
- J1 pad 15: /D4 -> (no net)
- J1 pad 16: /D6 -> (no net)
- J1 pad 17: Net-(J1-Pad17) -> (no net)
- J1 pad 18: Net-(J1-Pad18) -> (no net)
- J1 pad 19: Net-(J1-Pad19) -> (no net)
- J1 pad 2: /A0 -> (no net)
- J1 pad 20: Net-(J1-Pad20) -> (no net)
- J1 pad 21: Net-(J1-Pad21) -> (no net)
- J1 pad 22: Net-(J1-Pad22) -> (no net)
- J1 pad 23: /D7 -> (no net)
- J1 pad 24: /D5 -> (no net)
- J1 pad 25: /D3 -> (no net)
- J1 pad 26: /D1 -> (no net)
- J1 pad 27: Net-(J1-Pad27) -> (no net)
- J1 pad 28: Net-(J1-Pad28) -> (no net)
- J1 pad 29: Net-(J1-Pad29) -> (no net)
- J1 pad 3: /A1 -> (no net)
- J1 pad 30: Net-(J1-Pad30) -> (no net)
- J1 pad 31: Net-(J1-Pad31) -> (no net)
- J1 pad 32: Net-(J1-Pad32) -> (no net)
- J1 pad 33: Net-(J1-Pad33) -> (no net)
- J1 pad 34: Net-(J1-Pad34) -> (no net)
- J1 pad 35: Net-(J1-Pad35) -> (no net)
- J1 pad 36: Net-(J1-Pad36) -> (no net)
- J1 pad 4: /A0 -> (no net)
- J1 pad 5: /A5 -> (no net)
- J1 pad 6: /A6 -> (no net)
- J1 pad 7: /A7 -> (no net)
- J1 pad 8: /A8 -> (no net)
- J1 pad 9: /A9 -> (no net)
- J2 pad 1: Net-(J2-Pad1) -> (no net)
- J2 pad 12: /D0 -> (no net)
- J2 pad 13: /D1 -> (no net)
- J2 pad 14: /D2 -> (no net)
- J2 pad 15: Net-(J2-Pad15) -> (no net)
- J2 pad 16: Net-(J2-Pad16) -> (no net)
- J2 pad 17: Net-(J2-Pad17) -> (no net)
- J2 pad 18: Net-(J2-Pad18) -> (no net)
- J2 pad 19: Net-(J2-Pad19) -> (no net)
- J2 pad 2: Net-(J2-Pad2) -> (no net)
- J2 pad 20: Net-(J2-Pad20) -> (no net)
- J2 pad 21: Net-(J2-Pad21) -> (no net)
- J2 pad 22: /D3 -> (no net)
- J2 pad 23: /D4 -> (no net)
- J2 pad 24: /D5 -> (no net)
- J2 pad 25: /D6 -> (no net)
- J2 pad 26: /D7 -> (no net)
- J2 pad 27: Net-(J2-Pad27) -> (no net)
- J2 pad 28: Net-(J2-Pad28) -> (no net)
- J2 pad 29: Net-(J2-Pad29) -> (no net)
- J2 pad 3: Net-(J2-Pad3) -> (no net)
- J2 pad 30: Net-(J2-Pad30) -> (no net)
- J2 pad 31: Net-(J2-Pad31) -> (no net)
- J2 pad 32: Net-(J2-Pad32) -> (no net)
- J2 pad 33: Net-(J2-Pad33) -> (no net)
- J2 pad 34: Net-(J2-Pad34) -> (no net)
- J2 pad 35: Net-(J2-Pad35) -> (no net)
- J2 pad 36: Net-(J2-Pad36) -> (no net)
- J2 pad 4: /A7 -> (no net)
- J2 pad 5: /A6 -> (no net)
- J2 pad 6: /A5 -> (no net)
- K1 pad 1: Net-(K1-Pad1) -> (no net)
- K1 pad 2: Net-(K1-Pad2) -> (no net)
- K1 pad 3: Net-(K1-Pad3) -> (no net)
- K1 pad 4: Net-(K1-Pad4) -> (no net)
- K1 pad 5: Net-(K1-Pad5) -> (no net)
- R1 pad 1: Net-(R1-Pad1) -> (no net)
- R1 pad 2: Net-(R1-Pad2) -> (no net)
- U2 pad 1: Net-(U2-Pad1) -> (no net)
- U2 pad 2: Net-(U2-Pad2) -> (no net)
- U2 pad 3: Net-(U2-Pad3) -> (no net)
- U2 pad 4: Net-(U2-Pad4) -> (no net)
